Commit message: Fixed parser bugs, added info.txt, now IK solver is parsed as well

File: urdf/mk_root/mk_robot.xacro (robot description, xacro)
@@ -1,9 +1,9 @@
 <?xml version="1.0" ?>
-<robot name="trial2_robot" xmlns:xacro="http://www.ros.org/wiki/xacro">
+<robot name="mk_robot" xmlns:xacro="http://www.ros.org/wiki/xacro">
   <!--Constants for robot dimensions-->
   <xacro:property name="PI" value="3.1415926535897931"/>
   <xacro:property name="density" value="100.0"/>
   <xacro:property name="axel_offset" value="0.05"/>
-  <xacro:include filename="$(find robot_generator)/urdf/trial2_root/trial2_robot.gazebo"/>
+  <xacro:include filename="$(find robot_generator)/urdf/mk_root/mk_robot.gazebo"/>
   <xacro:include filename="$(find robot_generator)/urdf/materials.xacro"/>
   <!--World link for fixing robot to Gazebo frame-->
@@ -16,5 +16,5 @@
   <link name="link1">
     <collision>
-      <origin rpy="0 0 0" xyz="0 0 1.0"/>
+      <origin rpy="0 0 0" xyz="0 0 1"/>
       <geometry>
         <box size="0.1 0.1 2"/>
@@ -22,5 +22,5 @@
     </collision>
     <visual>
-      <origin rpy="0 0 0" xyz="0 0 1.0"/>
+      <origin rpy="0 0 0" xyz="0 0 1"/>
       <geometry>
         <box size="0.1 0.1 2"/>
@@ -29,5 +29,5 @@
     </visual>
     <inertial>
-      <origin rpy="0 0 0" xyz="0 0 1.0"/>
+      <origin rpy="0 0 0" xyz="0 0 1"/>
       <mass value="2.0"/>
       <inertia ixx="${2.0 / 12.0 * (0.1*0.1 + 2*2)}" ixy="0.0" ixz="0.0" iyy="${2.0 / 12.0 * (2*2 + 0.1*0.1)}" iyz="0.0" izz="${2.0 / 12.0 * (0.1*0.1 + 0.1*0.1)}"/>
@@ -73,20 +73,20 @@
   <link name="link3">
     <collision>
-      <origin rpy="0 0 0" xyz="0 0 ${0.5 - axel_offset}"/>
+      <origin rpy="0 0 0" xyz="0 0 ${0.25 - axel_offset}"/>
       <geometry>
-        <box size="0.1 0.1 1.0"/>
+        <box size="0.1 0.1 0.5"/>
       </geometry>
     </collision>
     <visual>
-      <origin rpy="0 0 0" xyz="0 0 ${0.5 - axel_offset}"/>
+      <origin rpy="0 0 0" xyz="0 0 ${0.25 - axel_offset}"/>
       <geometry>
-        <box size="0.1 0.1 1.0"/>
+        <box size="0.1 0.1 0.5"/>
       </geometry>
       <material name="orange"/>
     </visual>
     <inertial>
-      <origin rpy="0 0 0" xyz="0 0 ${0.5 - axel_offset}"/>
-      <mass value="1.0"/>
-      <inertia ixx="${1.0 / 12.0 * (0.1*0.1 + 1.0*1.0)}" ixy="0.0" ixz="0.0" iyy="${1.0 / 12.0 * (1.0*1.0 + 0.1*0.1)}" iyz="0.0" izz="${1.0 / 12.0 * (0.1*0.1 + 0.1*0.1)}"/>
+      <origin rpy="0 0 0" xyz="0 0 ${0.25 - axel_offset}"/>
+      <mass value="0.5"/>
+      <inertia ixx="${0.5 / 12.0 * (0.1*0.1 + 0.5*0.5)}" ixy="0.0" ixz="0.0" iyy="${0.5 / 12.0 * (0.5*0.5 + 0.1*0.1)}" iyz="0.0" izz="${0.5 / 12.0 * (0.1*0.1 + 0.1*0.1)}"/>
     </inertial>
   </link>
@@ -108,3 +108,40 @@
     </actuator>
   </transmission>
+  <link name="link4">
+    <collision>
+      <origin rpy="0 0 0" xyz="0 0 ${0.5 - axel_offset}"/>
+      <geometry>
+        <box size="0.1 0.1 1.0"/>
+      </geometry>
+    </collision>
+    <visual>
+      <origin rpy="0 0 0" xyz="0 0 ${0.5 - axel_offset}"/>
+      <geometry>
+        <box size="0.1 0.1 1.0"/>
+      </geometry>
+      <material name="black"/>
+    </visual>
+    <inertial>
+      <origin rpy="0 0 0" xyz="0 0 ${0.5 - axel_offset}"/>
+      <mass value="1.0"/>
+      <inertia ixx="${1.0 / 12.0 * (0.1*0.1 + 1.0*1.0)}" ixy="0.0" ixz="0.0" iyy="${1.0 / 12.0 * (1.0*1.0 + 0.1*0.1)}" iyz="0.0" izz="${1.0 / 12.0 * (0.1*0.1 + 0.1*0.1)}"/>
+    </inertial>
+  </link>
+  <joint name="joint3" type="continuous">
+    <parent link="link3"/>
+    <child link="link4"/>
+    <origin rpy="0 0 0" xyz="0 0.1 ${0.5 - axel_offset}"/>
+    <axis xyz="0 1 0"/>
+    <dynamics damping="0.7"/>
+  </joint>
+  <transmission name="tran3">
+    <type>transmission_interface/SimpleTransmission</type>
+    <joint name="joint3">
+      <hardwareInterface>hardware_interface/EffortJointInterface</hardwareInterface>
+    </joint>
+    <actuator name="motor3">
+      <hardwareInterface>hardware_interface/EffortJointInterface</hardwareInterface>
+      <mechanicalReduction>1</mechanicalReduction>
+    </actuator>
+  </transmission>
 </robot>
